Commit message: Add script to compile, add script to start,  modified README.md, merge parser in main node, remove unused packages, implement multi-robot support

File: src/ros_2d_multi_robot_simulator/urdf/simple_circle_robot.urdf (robot description, URDF)
Before this commit: robot simple_circle_robot, 1 links, 0 joints
Links:
- removed link pose
- added link robot_1; visual cylinder length=0.1 radius=1
